File: subsheets/europower.kicad_sch (KiCad schematic)
At the start: 4 parts

Commit message: adds cv input subsheet
Parts:
- gave numbers to parts that had none: 4
Changed lines of the file:
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@@
   (symbol (lib_id "kpm-jlcpcb-basic:1u C 0603") (at 104.14 86.614 0) (unit 1)
     (in_bom yes) (on_board yes) (dnp no) (fields_autoplaced)
-    (property "Reference" "C?" (at 102.87 80.264 0)
+    (property "Reference" "C1" (at 102.87 80.264 0)
       (effects (font (size 1.27 1.27)) hide)
     )
@@
     (instances
       (project "synth-subsheets"
-        (path "/a4893583-2878-4d86-bdba-6b18e8bd6cd6/0f719f49-af48-49d6-b383-27d2659056a0"
-          (reference "C?") (unit 1)
+        (path "/a4893583-2878-4d86-bdba-6b18e8bd6cd6/e925806b-6dc0-456c-811e-ed9c9aa1dfc9"
+          (reference "C1") (unit 1)
+        )
+        (path "/a4893583-2878-4d86-bdba-6b18e8bd6cd6/5f8583cd-ab79-4f24-93fb-2f203ed37297"
+          (reference "C4") (unit 1)
         )
       )
@@
     (instances
       (project "synth-subsheets"
-        (path "/a4893583-2878-4d86-bdba-6b18e8bd6cd6/0f719f49-af48-49d6-b383-27d2659056a0"
+        (path "/a4893583-2878-4d86-bdba-6b18e8bd6cd6/e925806b-6dc0-456c-811e-ed9c9aa1dfc9"
           (reference "#PWR08") (unit 1)
         )
+        (path "/a4893583-2878-4d86-bdba-6b18e8bd6cd6/5f8583cd-ab79-4f24-93fb-2f203ed37297"
+          (reference "#PWR0104") (unit 1)
+        )
       )
     )
@@
     (instances
       (project "synth-subsheets"
-        (path "/a4893583-2878-4d86-bdba-6b18e8bd6cd6/0f719f49-af48-49d6-b383-27d2659056a0"
+        (path "/a4893583-2878-4d86-bdba-6b18e8bd6cd6/e925806b-6dc0-456c-811e-ed9c9aa1dfc9"
           (reference "#PWR02") (unit 1)
         )
+        (path "/a4893583-2878-4d86-bdba-6b18e8bd6cd6/5f8583cd-ab79-4f24-93fb-2f203ed37297"
+          (reference "#PWR0101") (unit 1)
+        )
       )
     )
@@
     (instances
       (project "synth-subsheets"
-        (path "/a4893583-2878-4d86-bdba-6b18e8bd6cd6/0f719f49-af48-49d6-b383-27d2659056a0"
+        (path "/a4893583-2878-4d86-bdba-6b18e8bd6cd6/e925806b-6dc0-456c-811e-ed9c9aa1dfc9"
           (reference "#PWR09") (unit 1)
         )
+        (path "/a4893583-2878-4d86-bdba-6b18e8bd6cd6/5f8583cd-ab79-4f24-93fb-2f203ed37297"
+          (reference "#PWR0105") (unit 1)
+        )
       )
     )
@@
     (instances
       (project "synth-subsheets"
-        (path "/a4893583-2878-4d86-bdba-6b18e8bd6cd6/0f719f49-af48-49d6-b383-27d2659056a0"
+        (path "/a4893583-2878-4d86-bdba-6b18e8bd6cd6/e925806b-6dc0-456c-811e-ed9c9aa1dfc9"
           (reference "#PWR01") (unit 1)
         )
+        (path "/a4893583-2878-4d86-bdba-6b18e8bd6cd6/5f8583cd-ab79-4f24-93fb-2f203ed37297"
+          (reference "#PWR0102") (unit 1)
+        )
       )
     )
@@
     (instances
       (project "synth-subsheets"
-        (path "/a4893583-2878-4d86-bdba-6b18e8bd6cd6/0f719f49-af48-49d6-b383-27d2659056a0"
+        (path "/a4893583-2878-4d86-bdba-6b18e8bd6cd6/e925806b-6dc0-456c-811e-ed9c9aa1dfc9"
           (reference "#PWR06") (unit 1)
         )
+        (path "/a4893583-2878-4d86-bdba-6b18e8bd6cd6/5f8583cd-ab79-4f24-93fb-2f203ed37297"
+          (reference "#PWR0106") (unit 1)
+        )
       )
     )
@@
   (symbol (lib_id "kpm-jlcpcb-basic:1u C 0603") (at 106.426 99.06 0) (unit 1)
     (in_bom yes) (on_board yes) (dnp no) (fields_autoplaced)
-    (property "Reference" "C?" (at 105.156 92.71 0)
+    (property "Reference" "C2" (at 105.156 92.71 0)
       (effects (font (size 1.27 1.27)) hide)
     )
@@
     (instances
       (project "synth-subsheets"
-        (path "/a4893583-2878-4d86-bdba-6b18e8bd6cd6/0f719f49-af48-49d6-b383-27d2659056a0"
-          (reference "C?") (unit 1)
+        (path "/a4893583-2878-4d86-bdba-6b18e8bd6cd6/e925806b-6dc0-456c-811e-ed9c9aa1dfc9"
+          (reference "C2") (unit 1)
+        )
+        (path "/a4893583-2878-4d86-bdba-6b18e8bd6cd6/5f8583cd-ab79-4f24-93fb-2f203ed37297"
+          (reference "C5") (unit 1)
         )
       )
@@
     (instances
       (project "synth-subsheets"
-        (path "/a4893583-2878-4d86-bdba-6b18e8bd6cd6/0f719f49-af48-49d6-b383-27d2659056a0"
+        (path "/a4893583-2878-4d86-bdba-6b18e8bd6cd6/e925806b-6dc0-456c-811e-ed9c9aa1dfc9"
           (reference "#PWR03") (unit 1)
         )
+        (path "/a4893583-2878-4d86-bdba-6b18e8bd6cd6/5f8583cd-ab79-4f24-93fb-2f203ed37297"
+          (reference "#PWR0108") (unit 1)
+        )
       )
     )
@@
   (symbol (lib_id "EuroRackTools:EuroPower16") (at 148.336 86.614 0) (unit 1)
     (in_bom yes) (on_board yes) (dnp no) (fields_autoplaced)
-    (property "Reference" "J?" (at 149.606 76.2 0)
+    (property "Reference" "J2" (at 149.606 76.2 0)
       (effects (font (size 1.27 1.27)))
     )
@@
     (instances
       (project "synth-subsheets"
-        (path "/a4893583-2878-4d86-bdba-6b18e8bd6cd6/0f719f49-af48-49d6-b383-27d2659056a0"
-          (reference "J?") (unit 1)
+        (path "/a4893583-2878-4d86-bdba-6b18e8bd6cd6/e925806b-6dc0-456c-811e-ed9c9aa1dfc9"
+          (reference "J2") (unit 1)
+        )
+        (path "/a4893583-2878-4d86-bdba-6b18e8bd6cd6/5f8583cd-ab79-4f24-93fb-2f203ed37297"
+          (reference "J3") (unit 1)
         )
       )
@@
     (instances
       (project "synth-subsheets"
-        (path "/a4893583-2878-4d86-bdba-6b18e8bd6cd6/0f719f49-af48-49d6-b383-27d2659056a0"
+        (path "/a4893583-2878-4d86-bdba-6b18e8bd6cd6/e925806b-6dc0-456c-811e-ed9c9aa1dfc9"
           (reference "#PWR04") (unit 1)
         )
+        (path "/a4893583-2878-4d86-bdba-6b18e8bd6cd6/5f8583cd-ab79-4f24-93fb-2f203ed37297"
+          (reference "#PWR0109") (unit 1)
+        )
       )
     )
@@
   (symbol (lib_id "kpm-jlcpcb-basic:1u C 0603") (at 111.76 86.614 0) (unit 1)
     (in_bom yes) (on_board yes) (dnp no) (fields_autoplaced)
-    (property "Reference" "C?" (at 110.49 80.264 0)
+    (property "Reference" "C3" (at 110.49 80.264 0)
       (effects (font (size 1.27 1.27)) hide)
     )
@@
     (instances
       (project "synth-subsheets"
-        (path "/a4893583-2878-4d86-bdba-6b18e8bd6cd6/0f719f49-af48-49d6-b383-27d2659056a0"
-          (reference "C?") (unit 1)
+        (path "/a4893583-2878-4d86-bdba-6b18e8bd6cd6/e925806b-6dc0-456c-811e-ed9c9aa1dfc9"
+          (reference "C3") (unit 1)
+        )
+        (path "/a4893583-2878-4d86-bdba-6b18e8bd6cd6/5f8583cd-ab79-4f24-93fb-2f203ed37297"
+          (reference "C6") (unit 1)
         )
       )
@@
     (instances
       (project "synth-subsheets"
-        (path "/a4893583-2878-4d86-bdba-6b18e8bd6cd6/0f719f49-af48-49d6-b383-27d2659056a0"
+        (path "/a4893583-2878-4d86-bdba-6b18e8bd6cd6/e925806b-6dc0-456c-811e-ed9c9aa1dfc9"
           (reference "#PWR07") (unit 1)
         )
+        (path "/a4893583-2878-4d86-bdba-6b18e8bd6cd6/5f8583cd-ab79-4f24-93fb-2f203ed37297"
+          (reference "#PWR0107") (unit 1)
+        )
       )
     )
@@
     (instances
       (project "synth-subsheets"
-        (path "/a4893583-2878-4d86-bdba-6b18e8bd6cd6/0f719f49-af48-49d6-b383-27d2659056a0"
+        (path "/a4893583-2878-4d86-bdba-6b18e8bd6cd6/e925806b-6dc0-456c-811e-ed9c9aa1dfc9"
           (reference "#PWR05") (unit 1)
         )
-      )
+        (path "/a4893583-2878-4d86-bdba-6b18e8bd6cd6/5f8583cd-ab79-4f24-93fb-2f203ed37297"
+          (reference "#PWR0103") (unit 1)
+        )
+      )
